Commit message: urdf created,Gazebo Simulation with Rviz is done

File: description/robot.urdf.xacro (robot description, xacro)
@@ -3,3 +3,4 @@
   <!-- Include the robot_core.xacro file -->
   <xacro:include filename="$(find pi_bot_2)/description/robot_core.xacro" />
+  <xacro:include filename="$(find pi_bot_2)/description/gazebo_control.xacro" />
 </robot>

File: description/robot_core.xacro (robot description, xacro)
@@ -41,4 +41,7 @@
         </xacro:inertial_box>
     </link>
+    <!-- <gazebo reference="chassis">
+        <material>Gazebo/White</material>
+    </gazebo> -->
     <!-- LEFT WHEEL LINK -->
     <joint name="left_wheel_joint" type="continuous">
@@ -64,4 +67,7 @@
         </xacro:inertial_cylinder>
     </link>
+    <!-- <gazebo reference="left_wheel">
+        <material>Gazebo/Blue</material>
+    </gazebo> -->
     <!-- RIGHT WHEEL LINK -->
     <joint name="right_wheel_joint" type="continuous">
@@ -87,4 +93,7 @@
         </xacro:inertial_cylinder>
     </link>
+    <!-- <gazebo reference="right_wheel">
+        <material>Gazebo/Blue</material>
+    </gazebo> -->
     <!-- CASTER WHEEL LINK -->
     <joint name="caster_wheel_joint" type="fixed">
@@ -109,3 +118,17 @@
         </xacro:inertial_sphere>
     </link>
+    <gazebo reference="caster_wheel">
+        <material>Gazebo/Black</material>
+        <mu1 value="0.001"/>
+        <mu2 value="0.001"/>
+    </gazebo>
+    <gazebo reference="chassis">
+        <material>Gazebo/White</material>
+    </gazebo>
+    <gazebo reference="left_wheel">
+        <material>Gazebo/Yellow</material>
+    </gazebo> -->
+    <gazebo reference="right_wheel">
+        <material>Gazebo/Yellow</material>
+    </gazebo>
 </robot>
